Commit message: Uncommited changes

File: hardware/model/model.urdf (robot description, URDF)
Before this commit: robot truck, 7 links, 6 joints
Joints:
- removed joint front_left_wheel_steering
- removed joint front_right_wheel_steering
- removed joint rear_left_wheel_axle
- removed joint rear_right_wheel_axle
- added joint left_rear_axle: type continuous, parent base, child rear_left_wheel, origin xyz=-0.2025 0.11168 -0.01329, axis 0.0 1.0 0.0
- added joint left_steering_joint: type revolute, parent base, child front_left_cup, origin xyz=0.2025 0.10668 -0.01329, axis 0.0 0.0 1.0, limit lower=-0.69813 upper=0.5236 effort=30 velocity=1.0
- added joint right_rear_axle: type continuous, parent base, child rear_right_wheel, origin xyz=-0.2025 -0.11168 -0.01329, axis -0.0 1.0 -0.0
- added joint right_steering_joint: type revolute, parent base, child front_right_cup, origin xyz=0.2025 -0.10668 -0.01329, axis -0.0 -0.0 1.0, limit lower=-0.5236 upper=0.69813 effort=30 velocity=1.0
